File: TEENSY4.1/TEENSY4.1.kicad_sch (KiCad schematic)
At the start: 62 parts, among them J1 USB_B_Micro, J2 Micro_SD_Card, Q1 DMG2305UX, SW2 SW_Push, U1 TLV75733PDBV, U1(FLASH) W25Q32JVSS, U2 TPD3S014, U2(PSRAM) APS1604M-3SQRx-SN, U3 MKL02Z32VFG4, U4 W25Q32JVSS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

Commit message: Add files via upload
Added the footprints
Parts:
- added L1: 4.7 uH, Inductor_SMD:L_0805_2012Metric, symbol Device:L_Ferrite_Small
- C1, C2, C29, C3, C7: footprint (none) -> Capacitor_SMD:C_0603_1608Metric_Pad1.08x0.95mm_HandSolder
- C10, C15, C16, C17, C22, C24, C6, C9: footprint (none) -> Capacitor_SMD:C_0805_2012Metric_Pad1.18x1.45mm_HandSolder
- C11: footprint (none) -> Capacitor_SMD:CP_Elec_6.3x7.7
- C12, C13, C14, C18, C19, C20, C21, C23, C25, C26, C27, C28, C8: footprint (none) -> Capacitor_SMD:C_0402_1005Metric
- C30, C31, C32, C33, C4, C5: footprint (none) -> Capacitor_SMD:C_0603_1608Metric
- F1: footprint (none) -> Fuse:Fuse_1206_3216Metric
- FB1: footprint (none) -> Inductor_SMD:L_0805_2012Metric
- J1: footprint (none) -> Connector_USB:USB_Micro-B_Molex-105017-0001
- J2: footprint (none) -> Connector_Card:microSD_HC_Molex_104031-0811
- L2: renamed from L1; footprint (none) -> Inductor_SMD:L_0805_2012Metric
- L3: renamed from L2; footprint (none) -> Inductor_SMD:L_0805_2012Metric
- SW2: footprint (none) -> Button_Switch_THT:SW_PUSH_6mm
- Y1: footprint (none) -> Crystal:Crystal_SMD_3225-4Pin_3.2x2.5mm
- Y2: footprint (none) -> Crystal:Crystal_SMD_3215-2Pin_3.2x1.5mm
- renumbered U1(FLASH) to U1(FLASH)1, U2(PSRAM) to U2(PSRAM)1
Connections:
- net at C13.1, C14.1, C15.1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: now also L1.1
