File: Microcontroller_Board/Microcontroller_Board.kicad_sch (KiCad schematic)
At the start: 20 parts, among them J1 Conn_01x24_Socket, J2 Conn_01x24_Socket, J3 XT60-M, U1 SN65HVD230QDR, U2 DEV-16771, U3 LMR51450SDRRR

Commit message: Add files via upload
Parts:
- removed CANHL1: 2601-1102, symbol Connector:Conn_01x04_Pin
- removed ENC1: 2601-1104, symbol Connector:Conn_01x08_Pin
- removed J3: XT60-M, XT60-M:AMASS_XT60-M, symbol XT60-M:XT60-M
- added CANHL1, I2C1, J2, J3, J9: 2601-1102, CONN2_2601-1102_WAG, symbol wago_connectors:2601-1102
- added ENC1, ENC2, J1, J4, J5, J6, J7, J8, RLY1: 2601-1104, CONN4_2601-1104_WAG, symbol wago_connectors:2601-1104
- added R7, R8: 10k, symbol Device:R_US
- added X1: XT60-M, XT60-M:AMASS_XT60-M, symbol XT_connector:XT60-M
Connections:
- net 12V: now also X1.2 (POS)
- net 3.3V: now also J1.3 (Pin_3), J2.15 (Pin_15), U2.3.3V_2 (3.3V), U2.3.3V_3 (3.3V), ENC1.7 (4_1), ENC1.8 (4_2), ENC2.7 (4_1), ENC2.8 (4_2), J4.7 (4_1), J4.8 (4_2), R7.2, R8.2
- net 5V: now also J1.1 (Pin_1), U2.VIN
- net CAN_RX: now also J1.4 (Pin_4), U2.23 (A9)
- net CAN_TX: now also J1.5 (Pin_5), U2.22 (A8)
- net ENC1_A: now also J1.12 (Pin_12), U2.15 (A1), ENC1.5 (3_1), ENC1.6 (3_2)
- net ENC1_B: now also J1.13 (Pin_13), U2.14 (A0), ENC1.3 (2_1), ENC1.4 (2_2)
- net GND: now also ENC1.1 (1_1), ENC1.2 (1_2), ENC2.1 (1_1), ENC2.2 (1_2), X1.1 (NEG)
- net WAGO_CANH: now also CANHL1.1 (1_2)
- net WAGO_CANL: now also CANHL1.2 (2_2)
- net ST_POT: now reaches J1.10 (Pin_10), U2.17 (A3)
- net A2: now reaches J1.11 (Pin_11), U2.16 (A2)
- net SCK: now reaches J1.14 (Pin_14), U2.13 (SCK)
- net SCK: now also J6.3 (2_1), J6.4 (2_2)
- net A17: now reaches J1.16 (Pin_16), U2.41 (A17)
- net A17: now also J6.1 (1_1), J6.2 (1_2)
- net ENC2_A: now reaches J1.17 (Pin_17), U2.40 (A16)
- net ENC2_A: now also ENC2.5 (3_1), ENC2.6 (3_2)
- net ENC2_B: now reaches J1.18 (Pin_18), U2.39 (A15)
- net ENC2_B: now also ENC2.3 (2_1), ENC2.4 (2_2)
- net A14: now reaches J1.19 (Pin_19), U2.38 (A14)
- net A14: now also J7.3 (2_1), J7.4 (2_2)
- net CS3: now reaches J1.20 (Pin_20), U2.37 (CS3)
- net CS3: now also J7.1 (1_1), J7.2 (1_2)
- net CS2: now reaches J1.21 (Pin_21), U2.36 (CS2)
- net CS2: now also J8.7 (4_1), J8.8 (4_2)
- net TX8: now reaches J1.22 (Pin_22), U2.35 (TX8)
- net TX8: now also J8.5 (3_1), J8.6 (3_2)
- net LC2_DAT: now reaches J1.23 (Pin_23), U2.34 (RX8)
- net LC2_CLK: now reaches J1.24 (Pin_24), U2.33 (MCLK2)
- net LC2_CLK: now also J8.1 (1_1), J8.2 (1_2)
- net LC1_CLK: now reaches J1.6 (Pin_6), U2.21 (A7)
- net LC1_DAT: now reaches J1.7 (Pin_7), U2.20 (A6)
- net LC4_DAT: now reaches J1.8 (Pin_8), U2.19 (A5)
- net LC4_CLK: now reaches J1.9 (Pin_9), U2.18 (A4)
- net RX1: now reaches J2.2 (Pin_2), U2.0 (RX1)
- net RX1: now also J9.1 (1_2)
- net TX1: now reaches J2.3 (Pin_3), U2.1 (TX1)
- net TX1: now also J9.2 (2_2)
- net CS1: now reaches J2.12 (Pin_12), U2.10 (CS1)
- net CS1: now also J4.1 (1_1), J4.2 (1_2)
- net ACME: now reaches J2.13 (Pin_13), U2.11 (MOSI)
- net ACME: now also J4.3 (2_1), J4.4 (2_2)
- net MISO: now reaches J2.14 (Pin_14), U2.12 (MISO)
- net MISO: now also J4.5 (3_1), J4.6 (3_2)
- net RLYON: now reaches J2.4 (Pin_4), U2.2 (OUT2)
- net RLYON: now also RLY1.1 (1_1), RLY1.2 (1_2)
- net I2C_SCL: now reaches J2.16 (Pin_16), U2.24 (A10)
- net I2C_SCL: now also I2C1.1 (1_2), R7.1
- net I2C_SDA: now reaches J2.17 (Pin_17), U2.25 (A11)
- net I2C_SDA: now also I2C1.2 (2_2), R8.1
- net LC3_DAT: now reaches J2.18 (Pin_18), U2.26 (A12)
- net LC3_DAT: now also J1.5 (3_1), J1.6 (3_2)
- net LC3_CLK: now reaches J2.19 (Pin_19), U2.27 (A13)
- net LC3_CLK: now also J1.7 (4_1), J1.8 (4_2)
- net RX7: now reaches J2.20 (Pin_20), U2.28 (RX7)
- net RX7: now also J2.1 (1_2)
- net TX7: now reaches J2.21 (Pin_21), U2.29 (TX7)
- net TX7: now also J2.2 (2_2)
- net RLYGD: now reaches J2.5 (Pin_5), U2.3 (LRCLK2)
- net RLYGD: now also RLY1.3 (2_1), RLY1.4 (2_2)
- net CRX3: now reaches J2.22 (Pin_22), U2.30 (CRX3)
- net CRX3: now also J3.1 (1_2)
- net CTX3: now reaches J2.23 (Pin_23), U2.31 (CTX3)
- net CTX3: now also J3.2 (2_2)
- net OUT1B: now reaches J2.24 (Pin_24), U2.32 (OUT1B)
- net RLY3SL: now reaches J2.6 (Pin_6), U2.4 (BCLK2)
- net RLY3SL: now also RLY1.5 (3_1), RLY1.6 (3_2)
- net RLY6SL: now reaches J2.7 (Pin_7), U2.5 (IN2)
- net RLY6SL: now also RLY1.7 (4_1), RLY1.8 (4_2)
- net OUT1D: now reaches J2.8 (Pin_8), U2.6 (OUT1D)
- net OUT1D: now also J5.1 (1_1), J5.2 (1_2)
- net RX2: now reaches J2.9 (Pin_9), U2.7 (RX2)
- net RX2: now also J5.3 (2_1), J5.4 (2_2)
- net TX2: now reaches J2.10 (Pin_10), U2.8 (TX2)
- net TX2: now also J5.5 (3_1), J5.6 (3_2)
- net OUT1C: now reaches J2.11 (Pin_11), U2.9 (OUT1C)
- net OUT1C: now also J5.7 (4_1), J5.8 (4_2)
- new net ???: J1.1 (1_1), J1.2 (1_2), J1.3 (2_1), J1.4 (2_2), J6.5 (3_1), J6.6 (3_2), J6.7 (4_1), J6.8 (4_2), J7.5 (3_1), J7.6 (3_2), J7.7 (4_1), J7.8 (4_2)
- new net LCD_DAT: J8.3 (2_1), J8.4 (2_2)
Other:
- moved on the sheet: C1, C2, C3, C4, D2, J1, J2, L5.6H1, R1, R2, R3, R4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

Commit message: Add files via upload
Connections:
- net LCD_DAT is gone; now on net LC2_DAT: J8.3 (2_1), J8.4 (2_2)
- net RX2 is gone; now on net LC4_DAT: J2.9 (Pin_9), J5.3 (2_1), J5.4 (2_2), U2.7 (RX2)
- net RX7 is gone; now on net LC1_CLK: J2.1 (1_2), J2.20 (Pin_20), U2.28 (RX7)
- net TX2 is gone; now on net LC4_CLK: J2.10 (Pin_10), J5.5 (3_1), J5.6 (3_2), U2.8 (TX2)
- net TX7 is gone; now on net LC1_DAT: J2.2 (2_2), J2.21 (Pin_21), U2.29 (TX7)
- net A14: now also J6.7 (4_1), J6.8 (4_2); no longer J7.3 (2_1), J7.4 (2_2)
- net LC1_CLK: no longer J1.6 (Pin_6), U2.21 (A7)
- net LC1_DAT: no longer J1.7 (Pin_7), U2.20 (A6)
- net LC4_CLK: no longer J1.9 (Pin_9), U2.18 (A4)
- net LC4_DAT: no longer J1.8 (Pin_8), U2.19 (A5)
- net OUT1B: now also J6.5 (3_1), J6.6 (3_2)
- net ST_POT: now also J1.3 (2_1), J1.4 (2_2)
- removed net ???: J1.1 (1_1), J1.2 (1_2), J1.3 (2_1), J1.4 (2_2), J6.5 (3_1), J6.6 (3_2), J6.7 (4_1), J6.8 (4_2), J7.5 (3_1), J7.6 (3_2), J7.7 (4_1), J7.8 (4_2)
- new net A4: J1.1 (1_1), J1.2 (1_2), J1.9 (Pin_9), U2.18 (A4)
- new net A5: J1.8 (Pin_8), J7.7 (4_1), J7.8 (4_2), U2.19 (A5)
- new net A6: J1.7 (Pin_7), J7.5 (3_1), J7.6 (3_2), U2.20 (A6)
- new net A7: J1.6 (Pin_6), J7.3 (2_1), J7.4 (2_2), U2.21 (A7)
Changed lines of the file:
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@@
+	(wire
+		(pts
+			(xy 269.24 77.47) (xy 278.13 77.47)
+		)
+		(stroke
+			(width 0)
+			(type default)
+		)
+	)
 	(wire
 		(pts
@@
 	(wire
 		(pts
-			(xy 273.05 77.47) (xy 278.13 77.47)
-		)
-		(stroke
-			(width 0)
-			(type default)
-		)
-	)
-	(wire
-		(pts
 			(xy 104.14 254) (xy 104.14 262.89)
 		)
@@
 	(wire
 		(pts
-			(xy 144.78 149.86) (xy 151.13 149.86)
+			(xy 142.24 149.86) (xy 151.13 149.86)
 		)
 		(stroke
@@
 	(wire
 		(pts
-			(xy 144.78 144.78) (xy 151.13 144.78)
+			(xy 142.24 144.78) (xy 151.13 144.78)
 		)
 		(stroke
@@
 	(wire
 		(pts
-			(xy 273.05 82.55) (xy 278.13 82.55)
+			(xy 269.24 82.55) (xy 278.13 82.55)
 		)
 		(stroke
@@
 		)
 	)
-	(label "LC1_CLK"
+	(label "A7"
 		(at 369.57 182.88 0)
 		(effects
@@
 		)
 	)
-	(label "RX7"
-		(at 144.78 144.78 0)
+	(label "LC1_CLK"
+		(at 142.24 144.78 0)
 		(effects
 			(font
@@
 		)
 	)
-	(label "LC4_CLK"
+	(label "A4"
 		(at 369.57 190.5 0)
 		(effects
@@
 		)
 	)
-	(label "???"
+	(label "A6"
 		(at 190.5 83.82 0)
 		(effects
@@
 		)
 	)
-	(label "TX7"
-		(at 144.78 149.86 0)
+	(label "LC1_DAT"
+		(at 142.24 149.86 0)
 		(effects
 			(font
@@
 		)
 	)
-	(label "LC1_DAT"
+	(label "A6"
 		(at 369.57 185.42 0)
 		(effects
@@
 		)
 	)
-	(label "LCD_DAT"
+	(label "LC2_DAT"
 		(at 121.92 110.49 0)
 		(effects
@@
 		)
 	)
-	(label "TX2"
+	(label "LC4_CLK"
 		(at 285.75 180.34 0)
 		(effects
@@
 		)
 	)
-	(label "???"
+	(label "A14"
 		(at 220.98 90.17 0)
 		(effects
@@
 		)
 	)
-	(label "LC4_DAT"
+	(label "A5"
 		(at 369.57 187.96 0)
 		(effects
@@
 		)
 	)
-	(label "TX2"
-		(at 273.05 82.55 0)
-		(effects
-			(font
-				(size 1.27 1.27)
-			)
-			(justify left bottom)
-		)
-	)
-	(label "???"
+	(label "LC4_CLK"
+		(at 269.24 82.55 0)
+		(effects
+			(font
+				(size 1.27 1.27)
+			)
+			(justify left bottom)
+		)
+	)
+	(label "A5"
 		(at 190.5 88.9 0)
 		(effects
@@
 		)
 	)
-	(label "RX2"
+	(label "LC4_DAT"
 		(at 285.75 176.53 0)
 		(effects
@@
 		)
 	)
-	(label "A14"
+	(label "A7"
 		(at 190.5 78.74 0)
 		(effects
@@
 		)
 	)
-	(label "???"
+	(label "A4"
 		(at 99.06 142.24 0)
 		(effects
@@
 		)
 	)
-	(label "RX2"
-		(at 273.05 77.47 0)
-		(effects
-			(font
-				(size 1.27 1.27)
-			)
-			(justify left bottom)
-		)
-	)
-	(label "RX7"
+	(label "LC4_DAT"
+		(at 269.24 77.47 0)
+		(effects
+			(font
+				(size 1.27 1.27)
+			)
+			(justify left bottom)
+		)
+	)
+	(label "LC1_CLK"
 		(at 284.48 224.79 0)
 		(effects
@@
 		)
 	)
-	(label "TX7"
+	(label "LC1_DAT"
 		(at 284.48 229.87 0)
 		(effects
@@
 		)
 	)
-	(label "???"
+	(label "ST_POT"
 		(at 99.06 147.32 0)
 		(effects
@@
 		)
 	)
-	(label "???"
+	(label "OUT1B"
 		(at 220.98 85.09 0)
 		(effects

Commit message: Add files via upload
Parts:
- added X2: XT30P-M, XT30PW-M:AMASS_XT30PW-M, symbol XT_connector:XT30PW-M
Connections:
- net 5V: now also X2.2 (P)
- net GND: now also X2.1 (N)
Other:
- moved on the sheet: R7, R8
