File: Microcontroller_Board/Microcontroller_organized.kicad_sch (KiCad schematic)
At the start: 40 parts, among them J1 2601-1102, J2 2601-1104, J3 2601-1104, J4 2601-1104, J5 2601-1104, J6 2601-1104, J7 Conn_01x24_Socket, J8 Conn_01x24_Socket, J9 USB_A, U1 SN65HVD230QDR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

Commit message: Add files via upload
Parts:
- C1: value 0.1uF1 -> 100nF1; footprint Capacitor_SMD:C_0805_2012Metric -> Capacitor_SMD:C_0402_1005Metric_Pad0.74x0.62mm_HandSolder
- C2: value 10uF1 -> 10uF2; footprint Capacitor_SMD:C_0805_2012Metric_Pad1.18x1.45mm_HandSolder -> Capacitor_SMD:C_1206_3216Metric_Pad1.33x1.80mm_HandSolder
- C3: value 0.1uf2 -> 100nF2; footprint Capacitor_SMD:C_0805_2012Metric -> Capacitor_SMD:C_0402_1005Metric_Pad0.74x0.62mm_HandSolder
- C4: value 4.7uF1 -> 47uF3; footprint Capacitor_SMD:C_0805_2012Metric_Pad1.18x1.45mm_HandSolder -> Capacitor_SMD:C_1210_3225Metric_Pad1.33x2.70mm_HandSolder
- C5: value 4.7uF1 -> 47uF2; footprint Capacitor_SMD:C_0805_2012Metric_Pad1.18x1.45mm_HandSolder -> Capacitor_SMD:C_1210_3225Metric_Pad1.33x2.70mm_HandSolder
- C6: value 4.7uF1 -> 47uF1; footprint Capacitor_SMD:C_0805_2012Metric_Pad1.18x1.45mm_HandSolder -> Capacitor_SMD:C_1210_3225Metric_Pad1.33x2.70mm_HandSolder
- C7: footprint Capacitor_SMD:C_0805_2012Metric_Pad1.18x1.45mm_HandSolder -> Capacitor_SMD:C_1210_3225Metric_Pad1.33x2.70mm_HandSolder
Changed lines of the file:
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@@
 			)
 		)
-		(property "Value" "0.1uF1"
+		(property "Value" "100nF1"
 			(at 208.28 247.904 0)
 			(effects
@@
 			)
 		)
-		(property "Footprint" "Capacitor_SMD:C_0805_2012Metric"
+		(property "Footprint" "Capacitor_SMD:C_0402_1005Metric_Pad0.74x0.62mm_HandSolder"
 			(at 210.82 250.19 0)
 			(effects
@@
 			)
 		)
-		(property "Value" "0.1uf2"
+		(property "Value" "100nF2"
 			(at 133.35 244.094 0)
 			(effects
@@
 			)
 		)
-		(property "Footprint" "Capacitor_SMD:C_0805_2012Metric"
+		(property "Footprint" "Capacitor_SMD:C_0402_1005Metric_Pad0.74x0.62mm_HandSolder"
 			(at 135.89 246.38 0)
 			(effects
@@
 			)
 		)
-		(property "Footprint" "Capacitor_SMD:C_0805_2012Metric_Pad1.18x1.45mm_HandSolder"
+		(property "Footprint" "Capacitor_SMD:C_1210_3225Metric_Pad1.33x2.70mm_HandSolder"
 			(at 220.98 250.19 0)
 			(effects
@@
 			)
 		)
-		(property "Value" "4.7uF1"
+		(property "Value" "47uF3"
 			(at 99.06 250.444 0)
 			(effects
@@
 			)
 		)
-		(property "Footprint" "Capacitor_SMD:C_0805_2012Metric_Pad1.18x1.45mm_HandSolder"
+		(property "Footprint" "Capacitor_SMD:C_1210_3225Metric_Pad1.33x2.70mm_HandSolder"
 			(at 101.6 252.73 0)
 			(effects
@@
 			)
 		)
-		(property "Value" "10uF1"
+		(property "Value" "10uF2"
 			(at 229.87 247.904 0)
 			(effects
@@
 			)
 		)
-		(property "Footprint" "Capacitor_SMD:C_0805_2012Metric_Pad1.18x1.45mm_HandSolder"
+		(property "Footprint" "Capacitor_SMD:C_1206_3216Metric_Pad1.33x1.80mm_HandSolder"
 			(at 232.41 250.19 0)
 			(effects
@@
 			)
 		)
-		(property "Value" "4.7uF1"
+		(property "Value" "47uF1"
 			(at 72.39 250.444 0)
 			(effects
@@
 			)
 		)
-		(property "Footprint" "Capacitor_SMD:C_0805_2012Metric_Pad1.18x1.45mm_HandSolder"
+		(property "Footprint" "Capacitor_SMD:C_1210_3225Metric_Pad1.33x2.70mm_HandSolder"
 			(at 74.93 252.73 0)
 			(effects
@@
 			)
 		)
-		(property "Value" "4.7uF1"
+		(property "Value" "47uF2"
 			(at 86.36 250.444 0)
 			(effects
@@
 			)
 		)
-		(property "Footprint" "Capacitor_SMD:C_0805_2012Metric_Pad1.18x1.45mm_HandSolder"
+		(property "Footprint" "Capacitor_SMD:C_1210_3225Metric_Pad1.33x2.70mm_HandSolder"
 			(at 88.9 252.73 0)
 			(effects
