File: Microcontroller_Board/Microcontroller_organized.kicad_pcb (KiCad board)
At the start: 2 copper layers, 40 parts, among them J1 2601-1102, J2 2601-1104, J3 2601-1104, J4 2601-1104, J5 2601-1104, J6 2601-1104, J7 Conn_01x24_Socket, J8 Conn_01x24_Socket, J9 USB_A, U1 SN65HVD230QDR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

Commit message: finshied wiring pcb
Parts:
- moved C3 1.12 mm to (94.0, 86.5), turned to 90 degrees
- moved U3 0.25 mm to (97.0, 87.8)
- turned R3 to 0 degrees
- turned R9 to 180 degrees
Routing:
- net GND: track 81.7 -> 201.2 mm, vias 8 -> 12
- net /5V: track 3.96 -> 67.9 mm, vias 1 -> 5
- net /CAN_TX: track 3.91 -> 48.5 mm, vias 0 -> 2
- net /12V: track 3.83 -> 47.8 mm, vias 1 -> 5
- net /ENC1_B: track 9.43 -> 52.1 mm, vias 0 -> 2
- net /CAN_RX: track 3.91 -> 43.5 mm, vias 0 -> 4
- net /WAGO_CANL: track 5.40 -> 26.2 mm, vias 0 -> 2
- net /WAGO_CANH: track 5.00 -> 25.5 mm, vias 0 -> 2
- net Net-(J9-Shield): track 0.00 -> 17.6 mm
- net Net-(U1-RS): track 0.00 -> 16.5 mm, vias 0 -> 2
- net /3.3V: track 98.4 -> 111.5 mm, vias 3 -> 5
- net Net-(C3-Pad2): track 0.00 -> 8.45 mm, vias 0 -> 2
- net Net-(U3-FB): track 0.00 -> 5.31 mm
- net Net-(U3-ER): track 0.00 -> 2.70 mm
- net Net-(U3-BOOT): track 0.00 -> 2.44 mm
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
Commit message: Add files via upload
Parts:
- moved I2C1 2.50 mm to (160.0, 104.0)
- moved LC3&4 2.00 mm to (141.0, 104.0)
- moved C4 1.88 mm to (97.7, 83.7)
- moved R1 1.60 mm to (96.9, 74.4)
- moved J2 1.50 mm to (122.0, 104.0)
- moved C5 1.15 mm to (97.7, 77.1)
- moved CANHL1 1.00 mm to (81.0, 68.0)
- moved J1 1.00 mm to (110.0, 104.0)
- moved C6 0.83 mm to (97.7, 80.4)
- moved LC1&2 0.63 mm to (170.4, 104.8)
- moved RLY1 0.50 mm to (91.0, 104.0)
- moved C1 0.29 mm to (83.2, 112.8)
Routing:
- net /LC4_CLK: track 50.2 -> 10.8 mm
- net /LC4_DAT: track 36.7 -> 14.7 mm, vias 2 -> 1
- net /RLY6SL: track 38.0 -> 29.1 mm
- net GND: track 201.2 -> 194.3 mm
- net /5V: track 67.9 -> 63.2 mm
- net /SCK: track 27.5 -> 23.8 mm
- net /LC3_CLK: track 21.2 -> 18.1 mm
- net /I2C_SDA: track 84.6 -> 87.1 mm
- net /I2C_SCL: track 77.3 -> 79.8 mm
- net /CAN_RX: track 43.5 -> 45.9 mm
- net Net-(U1-RS): track 16.5 -> 15.6 mm, vias 2 -> 1
- net /LC3_DAT: track 18.7 -> 17.9 mm
- net /LC2_CLK: track 32.7 -> 33.4 mm
- net /OUT1D: track 16.1 -> 16.7 mm
- net /OUT1C: track 17.8 -> 17.2 mm
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