File: Microcontroller_Board/Microcontroller_organized.kicad_pcb (KiCad board)
At the start: 2 copper layers, 40 parts, among them J1 2601-1102, J2 2601-1104, J3 2601-1104, J4 2601-1104, J5 2601-1104, J6 2601-1104, J7 Conn_01x24_Socket, J8 Conn_01x24_Socket, J9 USB_A, U1 SN65HVD230QDR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

Commit message: shifted usb
Parts:
- moved J9 25.3 mm to (96.5, 109.2), turned to 0 degrees
- moved LC1&2 23.6 mm to (185.5, 86.7)
- moved J3 23.1 mm to (185.5, 68.9)
- moved I2C1 19.6 mm to (176.8, 94.0)
- moved RLY1 18.8 mm to (109.8, 104.1)
- moved LC3&4 18.7 mm to (159.7, 104.1)
- moved J1 18.6 mm to (128.6, 104.1)
- moved J2 18.3 mm to (140.3, 104.1)
Routing:
- net /LC4_CLK: track 10.8 -> 62.7 mm, vias 0 -> 2
- net /LC4_DAT: track 14.7 -> 53.9 mm, vias 1 -> 2
- net /CRX3: track 30.2 -> 68.7 mm, vias 2 -> 1
- net /MISO: track 45.9 -> 84.3 mm, vias 2 -> 0
- net /OUT1B: track 32.1 -> 70.3 mm, vias 2 -> 3
- net /3.3V: track 111.5 -> 79.0 mm, vias 5 -> 4
- net /CTX3: track 30.5 -> 59.7 mm
- net /I2C_SCL: track 79.8 -> 103.4 mm, vias 6 -> 2
- net /TX1: track 17.8 -> 37.7 mm
- net /LC1_DAT: track 26.2 -> 44.8 mm, vias 0 -> 1
- net /RLYGD: track 34.0 -> 16.0 mm
- net /RLYON: track 34.4 -> 16.4 mm
- net /RLY3SL: track 33.0 -> 15.9 mm
- net /RX1: track 17.7 -> 33.8 mm
- net /I2C_SDA: track 87.1 -> 103.0 mm, vias 6 -> 5
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- added copper zone on B.Cu, net GND
Other:
- board outline added: 130.7 x 65.7 mm
